File: pcb/gaggia-pid-pcb.kicad_sch (KiCad schematic)
At the start: 19 parts, among them J1 Conn_01x04, J2 Conn_01x02, J3 Conn_01x02, J4 Conn_01x02, U1 Adafruit MAX31865, U2 RP2040-ZERO

Commit message: Updated Vsens for PR2040-zero board
Parts:
- MH1, MH2, MH3, MH4: value M3 -> M2.5; footprint MountingHole:MountingHole_3.2mm_M3_Pad_Via -> MountingHole:MountingHole_2.7mm_M2.5_Pad_Via
Other:
- note added: "Power source connector (from AC/DC) approx +6V"
- note added: "Resistor choice based on stock I had. VDC scaling : 10k / 22k = 0.3125"
- note removed: "Power source connector (from AC/DC) ~ +6V"
- note removed: "Resistor choice based on stock I had. VDC scaling : 10k / 32k = 0.3125"
- moved on the sheet: MH1, MH2, MH3, MH4
Changed lines of the file:
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@@
 		)
 	)
-	(text "Resistor choice based on stock I had.\nVDC scaling : 10k / 32k = 0.3125"
+	(text "Resistor choice based on stock I had.\nVDC scaling : 10k / 22k = 0.3125"
 		(exclude_from_sim no)
 		(at 103.886 133.096 0)
@@
 		)
 	)
-	(text "Power source connector\n(from AC/DC) ~ +6V"
+	(text "Power source connector\n(from AC/DC) approx +6V"
 		(exclude_from_sim no)
 		(at 50.038 134.366 0)
@@
 	)
 	(junction
-		(at 49.53 186.69)
+		(at 48.26 186.69)
 		(diameter 0)
 		(color 0 0 0 0)
@@
 	)
 	(junction
-		(at 39.37 186.69)
+		(at 38.1 186.69)
 		(diameter 0)
 		(color 0 0 0 0)
 	)
 	(junction
-		(at 29.21 186.69)
+		(at 27.94 186.69)
 		(diameter 0)
 		(color 0 0 0 0)
@@
 	(wire
 		(pts
-			(xy 22.86 186.69) (xy 29.21 186.69)
+			(xy 22.86 186.69) (xy 27.94 186.69)
 		)
 		(stroke
@@
 	(wire
 		(pts
-			(xy 59.69 186.69) (xy 49.53 186.69)
+			(xy 58.42 186.69) (xy 48.26 186.69)
 		)
 		(stroke
@@
 	(wire
 		(pts
-			(xy 29.21 186.69) (xy 39.37 186.69)
+			(xy 27.94 186.69) (xy 38.1 186.69)
 		)
 		(stroke
@@
 	(wire
 		(pts
-			(xy 39.37 186.69) (xy 49.53 186.69)
+			(xy 38.1 186.69) (xy 48.26 186.69)
 		)
 		(stroke
@@
 	(symbol
 		(lib_id "Mechanical:MountingHole_Pad")
-		(at 29.21 184.15 0)
+		(at 27.94 184.15 0)
 		(unit 1)
 		(body_style 1)
@@
 		(fields_autoplaced yes)
 		(property "Reference" "MH1"
-			(at 31.75 181.6099 0)
+			(at 30.48 181.6099 0)
 			(show_name no)
 			(do_not_autoplace no)
@@
 			)
 		)
-		(property "Value" "M3"
-			(at 31.75 184.1499 0)
+		(property "Value" "M2.5"
+			(at 30.48 184.1499 0)
 			(show_name no)
 			(do_not_autoplace no)
@@
 			)
 		)
-		(property "Footprint" "MountingHole:MountingHole_3.2mm_M3_Pad_Via"
-			(at 29.21 184.15 0)
+		(property "Footprint" "MountingHole:MountingHole_2.7mm_M2.5_Pad_Via"
+			(at 27.94 184.15 0)
 			(hide yes)
 			(show_name no)
@@
 		)
 		(property "Datasheet" ""
-			(at 29.21 184.15 0)
+			(at 27.94 184.15 0)
 			(hide yes)
 			(show_name no)
@@
 		)
 		(property "Description" "Mounting Hole with connection"
-			(at 29.21 184.15 0)
+			(at 27.94 184.15 0)
 			(hide yes)
 			(show_name no)
@@
 		)
 		(property "Distributor Link 1" ""
-			(at 29.21 184.15 0)
+			(at 27.94 184.15 0)
 			(hide yes)
 			(show_name no)
@@
 		)
 		(property "Distributor Link 2" ""
-			(at 29.21 184.15 0)
+			(at 27.94 184.15 0)
 			(hide yes)
 			(show_name no)
@@
 		)
 		(property "LCSC" ""
-			(at 29.21 184.15 0)
+			(at 27.94 184.15 0)
 			(hide yes)
 			(show_name no)
@@
 		)
 		(property "Manufacturer Part Number" ""
-			(at 29.21 184.15 0)
+			(at 27.94 184.15 0)
 			(hide yes)
 			(show_name no)
@@
 	(symbol
 		(lib_id "Mechanical:MountingHole_Pad")
-		(at 59.69 184.15 0)
+		(at 58.42 184.15 0)
 		(unit 1)
 		(body_style 1)
@@
 		(fields_autoplaced yes)
 		(property "Reference" "MH4"
-			(at 62.23 181.6099 0)
+			(at 60.96 181.6099 0)
 			(show_name no)
 			(do_not_autoplace no)
@@
 			)
 		)
-		(property "Value" "M3"
-			(at 62.23 184.1499 0)
+		(property "Value" "M2.5"
+			(at 60.96 184.1499 0)
 			(show_name no)
 			(do_not_autoplace no)
@@
 			)
 		)
-		(property "Footprint" "MountingHole:MountingHole_3.2mm_M3_Pad_Via"
-			(at 59.69 184.15 0)
+		(property "Footprint" "MountingHole:MountingHole_2.7mm_M2.5_Pad_Via"
+			(at 58.42 184.15 0)
 			(hide yes)
 			(show_name no)
@@
 		)
 		(property "Datasheet" ""
-			(at 59.69 184.15 0)
+			(at 58.42 184.15 0)
 			(hide yes)
 			(show_name no)
@@
 		)
 		(property "Description" "Mounting Hole with connection"
-			(at 59.69 184.15 0)
+			(at 58.42 184.15 0)
 			(hide yes)
 			(show_name no)
@@
 		)
 		(property "Distributor Link 1" ""
-			(at 59.69 184.15 0)
+			(at 58.42 184.15 0)
 			(hide yes)
 			(show_name no)
@@
 		)
 		(property "Distributor Link 2" ""
-			(at 59.69 184.15 0)
+			(at 58.42 184.15 0)
 			(hide yes)
 			(show_name no)
@@
 		)
 		(property "LCSC" ""
-			(at 59.69 184.15 0)
+			(at 58.42 184.15 0)
 			(hide yes)
 			(show_name no)
@@
 		)
 		(property "Manufacturer Part Number" ""
-			(at 59.69 184.15 0)
+			(at 58.42 184.15 0)
 			(hide yes)
 			(show_name no)
@@
 	(symbol
 		(lib_id "Mechanical:MountingHole_Pad")
-		(at 39.37 184.15 0)
+		(at 38.1 184.15 0)
 		(unit 1)
 		(body_style 1)
@@
 		(fields_autoplaced yes)
 		(property "Reference" "MH2"
-			(at 41.91 181.6099 0)
+			(at 40.64 181.6099 0)
 			(show_name no)
 			(do_not_autoplace no)
@@
 			)
 		)
-		(property "Value" "M3"
-			(at 41.91 184.1499 0)
+		(property "Value" "M2.5"
+			(at 40.64 184.1499 0)
 			(show_name no)
 			(do_not_autoplace no)
@@
 			)
 		)
-		(property "Footprint" "MountingHole:MountingHole_3.2mm_M3_Pad_Via"
-			(at 39.37 184.15 0)
+		(property "Footprint" "MountingHole:MountingHole_2.7mm_M2.5_Pad_Via"
+			(at 38.1 184.15 0)
 			(hide yes)
 			(show_name no)
@@
 		)
 		(property "Datasheet" ""
-			(at 39.37 184.15 0)
+			(at 38.1 184.15 0)
 			(hide yes)
 			(show_name no)
@@
 		)
 		(property "Description" "Mounting Hole with connection"
-			(at 39.37 184.15 0)
+			(at 38.1 184.15 0)
 			(hide yes)
 			(show_name no)
@@
 		)
 		(property "Distributor Link 1" ""
-			(at 39.37 184.15 0)
+			(at 38.1 184.15 0)
 			(hide yes)
 			(show_name no)
@@
 		)
 		(property "Distributor Link 2" ""
-			(at 39.37 184.15 0)
+			(at 38.1 184.15 0)
 			(hide yes)
 			(show_name no)
@@
 		)
 		(property "LCSC" ""
-			(at 39.37 184.15 0)
+			(at 38.1 184.15 0)
 			(hide yes)
 			(show_name no)
@@
 		)
 		(property "Manufacturer Part Number" ""
-			(at 39.37 184.15 0)
+			(at 38.1 184.15 0)
 			(hide yes)
 			(show_name no)
@@
 	(symbol
 		(lib_id "Mechanical:MountingHole_Pad")
-		(at 49.53 184.15 0)
+		(at 48.26 184.15 0)
 		(unit 1)
 		(body_style 1)
@@
 		(fields_autoplaced yes)
 		(property "Reference" "MH3"
-			(at 52.07 181.6099 0)
+			(at 50.8 181.6099 0)
 			(show_name no)
 			(do_not_autoplace no)
@@
 			)
 		)
-		(property "Value" "M3"
-			(at 52.07 184.1499 0)
+		(property "Value" "M2.5"
+			(at 50.8 184.1499 0)
 			(show_name no)
 			(do_not_autoplace no)
@@
 			)
 		)
-		(property "Footprint" "MountingHole:MountingHole_3.2mm_M3_Pad_Via"
-			(at 49.53 184.15 0)
+		(property "Footprint" "MountingHole:MountingHole_2.7mm_M2.5_Pad_Via"
+			(at 48.26 184.15 0)
 			(hide yes)
 			(show_name no)
@@
 		)
 		(property "Datasheet" ""
-			(at 49.53 184.15 0)
+			(at 48.26 184.15 0)
 			(hide yes)
 			(show_name no)
@@
 		)
 		(property "Description" "Mounting Hole with connection"
-			(at 49.53 184.15 0)
+			(at 48.26 184.15 0)
 			(hide yes)
 			(show_name no)
@@
 		)
 		(property "Distributor Link 1" ""
-			(at 49.53 184.15 0)
+			(at 48.26 184.15 0)
 			(hide yes)
 			(show_name no)
@@
 		)
 		(property "Distributor Link 2" ""
-			(at 49.53 184.15 0)
+			(at 48.26 184.15 0)
 			(hide yes)
 			(show_name no)
@@
 		)
 		(property "LCSC" ""
-			(at 49.53 184.15 0)
+			(at 48.26 184.15 0)
 			(hide yes)
 			(show_name no)
@@
 		)
 		(property "Manufacturer Part Number" ""
-			(at 49.53 184.15 0)
+			(at 48.26 184.15 0)
 			(hide yes)
 			(show_name no)
